Commit message: Complete M3–M5: dual-source bridge, distribution monitor, risk engine, and HOC console. Add iiwa7 portfolio path, KL/MMD monitoring, React dashboard with WebSocket backend, experiment report export, docs assets, and verification scripts.

File: moveit_config/urdf/planar_2dof.urdf (robot description, URDF)
Before this commit: robot planar_2dof_arm, 4 links, 3 joints
Links:
- link base_link: mass 1.0 -> 2.0; geometry collision box size=0.14 0.14 0.44; collision box size=0.16 0.16 0.04
- link link1: geometry collision box size=0.30 0.06 0.06; visual box size=0.30 0.06 0.06
- link link2: geometry collision box size=0.25 0.05 0.05; visual box size=0.25 0.05 0.05
- link tool0: geometry collision sphere radius=0.035; visual sphere radius=0.035
Joints:
- joint ee_fixed_joint: origin xyz=0 0 0.125 rpy=0 0 0 -> xyz=0.25 0 0 rpy=0 0 0
- joint joint1: axis 0 0 1 -> 0 1 0; limit lower=-3.14 upper=3.14 effort=100 velocity=2.0 -> lower=-2.4 upper=2.4 effort=100 velocity=2.0; origin xyz=0 0 0.025 rpy=0 0 0 -> xyz=0 0 0.48 rpy=0 0 0
- joint joint2: axis 0 0 1 -> 0 1 0; origin xyz=0 0 0.15 rpy=0 0 0 -> xyz=0.30 0 0 rpy=0 0 0
